File: hardware/High Fructose.sch (EAGLE design)
At the start: 133 parts, among them U1 STM32F10XRXT6, U2 ADS1259, U3 ITG-3200, U4 MAX16903, U5 A4960, U6 A4960, U7 AH1804, X1 8MHz +/- 0.5%

Commit message: Update hardware dir with High Fructose
Parts:
- removed C29, C_HALL, C_MPU: 1uF, dan-rcl:C0603
- removed C30, C31, C32, C33, C34, C35, C36, C37, C38, C39, C40, C41, C42, C43, C44, C45, C46, C47, C48, C49, C50, C51, C52, C53, C54, C55, C56, C57, C58, C59, C60, C61, C62, C63, C64, C65, C66, C67, C68, C69, C70, C71, C72, C73: 22uF/16V, dan-rcl:C1206
- removed FB1, FB2: (no value), dan-rcl:FERRITE0603
- removed IC1: (no value), dan-vreg:MCP1826S
- removed JP3: (no value), pinhead:PINHD-1X1
- removed LDBT, LEDB, LEDY: (no value), dan-led:LED0805
- removed R11, R13, R9: 40mR/3W, rcl:R-US_R2512
- removed R12: 22k, dan-rcl:R0603
- removed R5: 330R, dan-rcl:R0603
- removed R6: 120k, dan-rcl:R0603
- removed S10, S11, S12, S7, S8, S9: MOSFET-N56, xow:MOSFET-N56
- removed TP1, TP2, TP4, TP5, TP6: TPB1,27, testpad:TPB1,27
- removed U$1: ADXRSXXXSMD, SparkFun-Sensors:ADXRSXXXSMD
- removed U$2: BLUETOOTH-RN41", SparkFun-RF:BLUETOOTH-RN41"
- added J1: JTAG-MINI, xow:JTAG-MINI
- added LEDP, LEDQ, LEDR: (no value), dan-led:LED0805
- added SW1: B3U-1000P, xow:SWITCH_SPST-NOB3U-1000P
- C1: value 22uF/16V -> 10uF/16V
- C10, C11, C12, C14, C27, C28: value 1uF -> 22uF/16V; device dan-rcl:C0603 -> dan-rcl:C1206
- C13: value 2.2nF -> 22uF/16V; device dan-rcl:C0603 -> dan-rcl:C1206
- C22: value 0.47uF/16V -> 22uF/16V; device dan-rcl:C0603 -> dan-rcl:C1206
- C23: value 10uF/16V -> 22uF/16V; device dan-rcl:C0805 -> dan-rcl:C1206
- C24, C25, C26: value 0.1uF/16V -> 22uF/16V; device dan-rcl:C0603 -> dan-rcl:C1206
- C4: value 22uF -> 10nF; device dan-rcl:C0805 -> dan-rcl:C0603
- C6: value 22nF -> 0.47uF
- C7: value 22nF -> 22uF; device dan-rcl:C0603 -> dan-rcl:C0805
- C8: value 2.2nF -> 10uF
- JP1: device pinhead:PINHD-1X1 -> pinhead-2:PINHD-1X03_2.54-S
- JP2: device pinhead:PINHD-1X1 -> pinhead-2:PINHD-1X04_2.54-S
- L1: value 10uH -> 4.7uH
- R4: value 180R -> 10k
- R8: value 40mR/3W -> 10mR/3W
- U2: value ADS1259 -> L3G4200D; device xow:ADS1259 -> SparkFun-Sensors:L3G4200D
- U3: value ITG-3200 -> VNH5050A; device SparkFun-Sensors:ITG-3200 -> Xo-PowerIC:VNH5050A
- U6: value A4960 -> VNH5050A; device xow:A4960 -> Xo-PowerIC:VNH5050A
- U7: value AH1804 -> AS1362; device xow:AH1804 -> Xo-VReg:AS1362
Connections:
- removed net ADC_MISO: U1PORTA_L.PA6, U2.DOUT
- removed net ADC_MOSI: U1PORTA_L.PA7, U2.DIN
- removed net ADC_NSS: U1PORTA_L.PA4, U2.!CS
- removed net ADC_SCK: U1PORTA_L.PA5, U2.SCLK
- removed net AGND: C11.2, C27.2, C28.2, C29.2, C8.1, FB1.1, U$1.AGND, U$1.PGND, U2.AVSS
- removed net BT_CTS: U$2.UARTRTS, U1PORTA_L.PA0
- removed net BT_RTS: U$2.UARTCTS, U1PORTA_L.PA1
- removed net BT_RX: U$2.UARTTX, U1PORTA_L.PA3
- removed net BT_TX: U$2.UARTRX, U1PORTA_L.PA2
- removed net HALL: U1PORTB_L.PB3, U7.OUT
- removed net LED1: R2.2, U1PORTB_L.PB0
- removed net LED2: R3.2, U1PORTB_H.PB10
- removed net LEDB: R1.2, U1PORTC_L.PC4
- removed net LEDY: R4.2, U1PORTB_H.PB12
- removed net M2_A: C24.2, S7.S, S8.D, U6.SA
- removed net M2_B: C25.2, S10.D, S9.S, U6.SB
- removed net M2_C: C26.2, S11.S, S12.D, U6.SC
- removed net M2_DIAG: U1PORTC_L.PC7, U6.DIAG
- removed net M2_LSS: R11.2, R13.2, S10.S, S12.S, S8.S, U6.CSP, U6.LSS
- removed net M2_MISO: U1PORTC_H.PC11, U6.SDO
- removed net M2_MOSI: U1PORTC_H.PC12, U6.SDI
- removed net M2_NSS: U1PORTD/OSC.PD2, U6.STRN
- removed net M2_PWM: U1PORTC_H.PC8, U6.PWM
- removed net M2_SCK: U1PORTC_H.PC10, U6.SCK
- removed net M2_TACHO: U1PORTA_H.PA15, U6.TACHO
- removed net MPU_SCL: U1PORTB_H.PB8, U3.SCL
- removed net MPU_SDA: U1PORTB_L.PB7, U3.SDA
- removed net N$10: C6.1, U$1.CP2
- removed net N$12: C7.1, U$1.CP4
- removed net N$13: C8.2, U$1.CP5
- removed net N$14: C9.1, R6.1, U$1.RATEOUT, U2.AINP
- removed net N$15: C9.2, R6.2, U$1.SUMJ
- removed net N$16: C11.1, U2.AINN, U2.REFOUT
- removed net N$17: C10.2, U2.VREFN
- removed net N$18: C10.1, U2.VREFP
- removed net N$19: C12.1, U2.BYPASS
- removed net N$20: C13.2, U3.CPOUT
- removed net N$21: C14.2, U3.REGOUT
- removed net N$23: C3.1, FB2.2, L1.1
- removed net N$32: R5.2, U$2.PIO5
- removed net N$33: LDBT.A, R5.1
- removed net N$34: C22.2, U6.CP2
- removed net N$36: C22.1, U6.CP1
- removed net N$47: C23.1, U6.VREG
- removed net N$50: S7.G, U6.GHA
- removed net N$51: S8.G, U6.GLA
- removed net N$52: C24.1, U6.CA
- removed net N$54: S9.G, U6.GHB
- removed net N$55: S10.G, U6.GLB
- removed net N$56: C25.1, U6.CB
- removed net N$57: S11.G, U6.GHC
- removed net N$59: S12.G, U6.GLC
- removed net N$60: C26.1, U6.CC
- removed net N$62: R12.1, U6.RESETN
- removed net U1_RX: TP2.TP, U1PORTA_H.PA10
- removed net U1_TX: TP1.TP, U1PORTA_H.PA9
- new net +UB: C10.1, C11.1, C12.1, C13.1, C14.1, C22.1, C23.1, R10.2, S1.D, S3.D, S5.D, U5.VBB, U5.VBRG
- new net -UB: C10.2, C11.2, C12.2, C13.2, C14.2, C22.2, C23.2, R8.1, U5.CSM
- new net BUT1: SW1.2, U1PORTC_H.PC13
- new net GYRO_SCL: U1PORTB_H.PB8, U2.SCL
- new net GYRO_SDA: U1PORTB_L.PB7, U2.SDA/SDI
- new net LEDP: R3.2, U1PORTA_L.PA1
- new net LEDQ: R1.2, U1PORTA_L.PA2
- new net LEDR: R2.2, U1PORTA_L.PA3
- new net MTR_A: U1PORTC_H.PC9, U6.INB
- new net MTR_B: U1PORTA_H.PA9, U6.INA
- new net MTR_EN: U1PORTB_H.PB12, U3.CS_DIS, U3.ENA/DIAGA, U3.ENB/DIAGB, U6.CS_DIS, U6.ENA/DIAGA, U6.ENB/DIAGB
- new net MTR_X: U1PORTA_H.PA10, U3.INB
- new net MTR_Y: U1PORTA_H.PA12, U3.INA
- new net M_A: U6.OUTB
- new net M_B: U6.OUTA
- new net M_X: U3.OUTB
- new net M_Y: U3.OUTA
- new net PWM_AB: U1PORTA_H.PA8, U6.IN_PWM
- new net PWM_XY: U1PORTA_H.PA11, U3.IN_PWM
- new net RX_PPM: JP1.3, U1PORTA_H.PA15
- new net SWO: J1.TDO/SWO, U1PORTB_L.PB3
- new net UART_RX: JP2.4, U1PORTC_L.PC7
- new net UART_TX: JP2.3, U1PORTC_L.PC6
- net !RESET: now also J1.NRST, U7.POK; no longer TP6.TP
- net +5V: now also C3.1, JP1.2, L1.1, U7.!SHDN, U7.IN; no longer C27.1, C28.1, C29.1, C4.1, FB2.1, IC1.IN, U$1.AVCC, U$1.VDD, U$1.VRATIO, U2.AVDD
- net GND: now also C4.2, C6.2, C7.2, C8.2, J1.GND, JP1.1, LEDP.C, LEDQ.C, LEDR.C, SW1.1, U2.GND, U2.RSDVG@3, U2.RSVDG@0, U2.RSVDG@1, U2.RSVDG@2, U2.RSVDG@4; no longer C12.2, C13.1, C14.1, C23.2, C_HALL.2, C_MPU.1, FB1.2, IC1.GND@2, IC1.GND@TAB, LEDB.C, LEDY.C, U$2.GND, U$2.GND1, U$2.GND4, U$2.GND5, U2.DGND, U2.START, U2.XTAL1, U3.AD0, U3.CLKIN, U3.GND, U3.RESV-G, U4.SYNC, U6.AGND, U6.GND
- net M1_LSS: no longer R9.2
- net M1_NSS: now also U1PORTC_H.PC8; no longer U1PORTC_L.PC6
- net N$11: now also LEDP.A, R3.1; no longer C7.2, U$1.CP3
- net N$28: now also U4.SYNC
- net N$35: now also LEDR.A, R2.1; no longer LEDY.A, R4.1
- net N$5: now also LEDQ.A; no longer LEDB.A
- net N$6: now also C4.1, R4.1, U2.PLL; no longer JP1.1, R3.1
- net N$7: now also C6.1, R4.2; no longer JP3.1, R2.1
- net N$9: now also C9.1, U7.BYPASS; no longer C6.2, U$1.CP1
- net SWCLK: now also J1.TCK/SWCLK; no longer TP4.TP
- net SWDIO: now also J1.TMS/SWDIO; no longer TP5.TP
- net V+: now also C24.1, C25.1, C26.1, C27.1, C28.1, U3.VCC, U6.VCC; no longer C30.1, C31.1, C32.1, C33.1, C34.1, C35.1, C36.1, C37.1, C38.1, C39.1, C40.1, C41.1, C42.1, C43.1, C44.1, C45.1, C46.1, C47.1, C48.1, C49.1, C50.1, C51.1, C52.1, C53.1, C54.1, C55.1, C56.1, C57.1, C58.1, C59.1, C60.1, C61.1, C62.1, C63.1, C64.1, C65.1, C66.1, C67.1, C68.1, C69.1, C70.1, C71.1, C72.1, C73.1, R10.2, R12.2, S1.D, S11.D, S3.D, S5.D, S7.D, S9.D, U5.VBB, U5.VBRG, U6.VBB, U6.VBRG
- net V-: now also C24.2, C25.2, C26.2, C27.2, C28.2, U3.GND_A, U3.GND_B, U6.GND_A, U6.GND_B; no longer C30.2, C31.2, C32.2, C33.2, C34.2, C35.2, C36.2, C37.2, C38.2, C39.2, C4.2, C40.2, C41.2, C42.2, C43.2, C44.2, C45.2, C46.2, C47.2, C48.2, C49.2, C50.2, C51.2, C52.2, C53.2, C54.2, C55.2, C56.2, C57.2, C58.2, C59.2, C60.2, C61.2, C62.2, C63.2, C64.2, C65.2, C66.2, C67.2, C68.2, C69.2, C70.2, C71.2, C72.2, C73.2, R11.1, R13.1, R8.1, R9.1, U5.CSM, U6.CSM
- net VDD: now also C7.1, C8.1, C9.2, J1.VDD, JP2.2, U2.CS, U2.RSVDV@0, U2.SDO, U2.VDD, U2.VDDIO, U7.OUT; no longer C_HALL.1, C_MPU.2, IC1.OUT, LDBT.C, U$2.VDD, U2.DVDD, U3.VDD, U3.VLOGIC, U6.REF, U6.VDD, U7.VDD
Other:
- note removed: "Bandwidth: 221Hz"
